File: Hardware/SparkFun_Pro_Mini-ESP32.kicad_pcb (KiCad board)
At the start: 2 copper layers, 33 x 17.8 mm, 76 parts, among them J1 Conn_01x06, J2 Conn_01x12, J3 Conn_01x12, J4 Qwiic_RA, SW1 Reset, SW2 Boot, U1 ESP32-PICO-V3-02, U2 AP2112K-3.3

Commit message: Update status LED to green.
Parts:
- D1: value Red -> Green
Changed lines of the file:
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@@
     (at 146.812 123.19 90)
     (tags "LED")
-    (property "PROD_ID" "DIO-00819")
+    (property "PROD_ID" "DIO-00821")
     (property "Sheetfile" "SparkFun_Pro_Mini-ESP32.kicad_sch")
     (property "Sheetname" "")
@@
         (effects (font (size 0.5 0.5) (thickness 0.1)))
     )
-    (fp_text value "Red" (at 0 1.43 90) (layer "F.Fab")
+    (fp_text value "Green" (at 0 1.43 90) (layer "F.Fab")
         (effects (font (size 0.5 0.5) (thickness 0.1)))
     )
